File: kicad/cocobuf.sch (KiCad schematic (older format))
At the start: 13 parts, among them P1 COCOBUS, U2 74LVC164245, U3 74LVC164245

Commit message: start of integration of common bus into CPLD
Parts:
- added D3: C_PWR, symbol LED
- added R3: 47K, symbol R
- added R4: 330, symbol R
Connections:
- net labels added: E
- net labels removed: ECLK
- wire segments 40 -> 43
Changed lines of the file:
@@
-EESchema Schematic File Version 2  date 4/22/2013 8:21:37 PM
+EESchema Schematic File Version 2  date 5/4/2013 9:22:42 PM
 LIBS:power
 LIBS:device
@@
 $Descr User 14000 8500
 encoding utf-8
-Sheet 3 3
+Sheet 3 4
 Title "Color Computer Bus Interface"
-Date "23 apr 2013"
-Rev "1.2"
-Comp "Bexkat Systems LLC"
+Date "5 may 2013"
+Rev "1.3"
+Comp "Bexkat Systems LLC 2013"
 Comment1 ""
 Comment2 ""
@@
 Comment4 ""
 $EndDescr
+Wire Wire Line
+	2950 3250 2950 3200
+Wire Wire Line
+	2950 3200 2900 3200
+Wire Wire Line
+	10050 6350 5550 6350
+Wire Wire Line
+	7450 4450 7450 4350
+Connection ~ 8050 4350
+Wire Wire Line
+	8050 4350 8050 4500
+Wire Wire Line
+	8100 4350 8100 4300
+Wire Wire Line
+	8350 4350 7850 4350
+Connection ~ 8100 4350
+Wire Wire Line
+	8150 4500 8150 4350
+Connection ~ 8150 4350
+Wire Wire Line
+	8750 4350 8750 4450
+Wire Wire Line
+	7350 1450 7350 1350
+Connection ~ 7950 1350
+Wire Wire Line
+	7950 1350 7950 1500
+Wire Wire Line
+	8000 1350 8000 1300
+Wire Wire Line
+	8250 1350 7750 1350
+Connection ~ 8000 1350
+Wire Wire Line
+	8050 1500 8050 1350
+Connection ~ 8050 1350
+Wire Wire Line
+	8650 1350 8650 1450
+Wire Wire Line
+	3650 3600 3650 3500
+Connection ~ 4250 3500
+Wire Wire Line
+	4250 3500 4250 3650
+Wire Wire Line
+	4300 3500 4300 3450
+Wire Wire Line
+	4550 3500 4050 3500
+Connection ~ 4300 3500
+Wire Wire Line
+	4350 3650 4350 3500
+Connection ~ 4350 3500
+Wire Wire Line
+	4950 3500 4950 3600
+Wire Wire Line
+	4900 1500 4900 1600
+Connection ~ 4300 1500
+Wire Wire Line
+	4300 1650 4300 1500
+Connection ~ 4250 1500
+Wire Wire Line
+	4500 1500 4000 1500
+Connection ~ 2250 2500
+Wire Wire Line
+	9200 6350 9200 5650
+Connection ~ 5550 4800
+Wire Wire Line
+	5550 6350 5550 2800
+Wire Wire Line
+	5550 4800 4900 4800
+Wire Wire Line
+	5550 2800 4850 2800
+Wire Wire Line
+	1600 2500 2250 2500
+Wire Wire Line
+	1950 5050 1950 4900
+Wire Wire Line
+	1950 4900 1600 4900
+Wire Wire Line
+	1950 5000 1600 5000
+Connection ~ 1950 5000
+Wire Wire Line
+	2650 2500 2650 2450
+Wire Wire Line
+	7500 5650 7500 5700
+Wire Wire Line
+	3700 4800 3700 4850
+Wire Wire Line
+	3650 2850 3650 2800
+Wire Wire Line
+	2250 2500 2250 2700
+Wire Wire Line
+	9200 5650 8700 5650
+Connection ~ 9200 6350
+Wire Wire Line
+	4250 1500 4250 1450
+Wire Wire Line
+	4200 1500 4200 1650
+Connection ~ 4200 1500
+Wire Wire Line
+	3600 1600 3600 1500
+Wire Wire Line
+	8700 5250 9050 5250
+Wire Wire Line
+	2250 2700 2750 2700
+Connection ~ 2500 2700
+$Comp
+L GND #PWR024
+U 1 1 517C6082
+P 2950 3250
+F 0 "#PWR024" H 2950 3250 30  0001 C CNN
+F 1 "GND" H 2950 3180 30  0001 C CNN
+	1    2950 3250
+	1    0    0    -1
+$EndComp
+$Comp
+L LED D3
+U 1 1 517C6080
+P 2700 3200
+F 0 "D3" H 2700 3300 50  0000 C CNN
+F 1 "C_PWR" H 2700 3100 50  0000 C CNN
+	1    2700 3200
+	1    0    0    -1
+$EndComp
+$Comp
+L R R4
+U 1 1 517C607E
+P 2500 2950
+F 0 "R4" V 2580 2950 50  0000 C CNN
+F 1 "330" V 2500 2950 50  0000 C CNN
+	1    2500 2950
+	1    0    0    -1
+$EndComp
+$Comp
+L GND #PWR025
+U 1 1 517C5438
+P 2250 3200
+F 0 "#PWR025" H 2250 3200 30  0001 C CNN
+F 1 "GND" H 2250 3130 30  0001 C CNN
+	1    2250 3200
+	1    0    0    -1
+$EndComp
+$Comp
+L R R3
+U 1 1 517C5423
+P 2250 2950
+F 0 "R3" V 2330 2950 50  0000 C CNN
+F 1 "47K" V 2250 2950 50  0000 C CNN
+	1    2250 2950
+	-1   0    0    1
+$EndComp
 NoConn ~ 4900 4700
 NoConn ~ 3700 4700
 NoConn ~ 1600 5400
-Wire Wire Line
-	10050 6350 5550 6350
-Wire Wire Line
-	7450 4450 7450 4350
-Connection ~ 8050 4350
-Wire Wire Line
-	8050 4350 8050 4500
-Wire Wire Line
-	8100 4350 8100 4300
-Wire Wire Line
-	8350 4350 7850 4350
-Connection ~ 8100 4350
-Wire Wire Line
-	8150 4500 8150 4350
-Connection ~ 8150 4350
-Wire Wire Line
-	8750 4350 8750 4450
-Wire Wire Line
-	7350 1450 7350 1350
-Connection ~ 7950 1350
-Wire Wire Line
-	7950 1350 7950 1500
-Wire Wire Line
-	8000 1350 8000 1300
-Wire Wire Line
-	8250 1350 7750 1350
-Connection ~ 8000 1350
-Wire Wire Line
-	8050 1500 8050 1350
-Connection ~ 8050 1350
-Wire Wire Line
-	8650 1350 8650 1450
-Wire Wire Line
-	3650 3600 3650 3500
-Connection ~ 4250 3500
-Wire Wire Line
-	4250 3500 4250 3650
-Wire Wire Line
-	4300 3500 4300 3450
-Wire Wire Line
-	4550 3500 4050 3500
-Connection ~ 4300 3500
-Wire Wire Line
-	4350 3650 4350 3500
-Connection ~ 4350 3500
-Wire Wire Line
-	4950 3500 4950 3600
-Wire Wire Line
-	4900 1500 4900 1600
-Connection ~ 4300 1500
-Wire Wire Line
-	4300 1650 4300 1500
-Connection ~ 4250 1500
-Wire Wire Line
-	4500 1500 4000 1500
-Connection ~ 2250 2500
-Wire Wire Line
-	9200 6350 9200 5650
-Connection ~ 5550 4800
-Wire Wire Line
-	5550 6350 5550 2800
-Wire Wire Line
-	5550 4800 4900 4800
-Wire Wire Line
-	5550 2800 4850 2800
-Wire Wire Line
-	1600 2500 2250 2500
-Wire Wire Line
-	1950 5050 1950 4900
-Wire Wire Line
-	1950 4900 1600 4900
-Wire Wire Line
-	1950 5000 1600 5000
-Connection ~ 1950 5000
-Wire Wire Line
-	2650 2500 2650 2450
-Wire Wire Line
-	7500 5650 7500 5700
-Wire Wire Line
-	3700 4800 3700 4850
-Wire Wire Line
-	3650 2850 3650 2800
-Wire Wire Line
-	2250 2500 2250 2700
-Wire Wire Line
-	9200 5650 8700 5650
-Connection ~ 9200 6350
-Wire Wire Line
-	4250 1500 4250 1450
-Wire Wire Line
-	4200 1500 4200 1650
-Connection ~ 4200 1500
-Wire Wire Line
-	3600 1600 3600 1500
-Wire Wire Line
-	8700 5250 9050 5250
 Text Label 9050 5250 0    60   ~ 0
 C_~SLENB
@@
 C_~SLENB
 $Comp
-L +3.3V #PWR029
+L +3.3V #PWR026
 U 1 1 5172867B
 P 8100 4300
-F 0 "#PWR029" H 8100 4260 30  0001 C CNN
+F 0 "#PWR026" H 8100 4260 30  0001 C CNN
 F 1 "+3.3V" H 8100 4410 30  0000 C CNN
 	1    8100 4300
@@
 $EndComp
 $Comp
-L GND #PWR030
+L GND #PWR027
 U 1 1 51728678
 P 7450 4450
-F 0 "#PWR030" H 7450 4450 30  0001 C CNN
+F 0 "#PWR027" H 7450 4450 30  0001 C CNN
 F 1 "GND" H 7450 4380 30  0001 C CNN
 	1    7450 4450
@@
 $EndComp
 $Comp
-L GND #PWR031
+L GND #PWR028
 U 1 1 51728677
 P 8750 4450
-F 0 "#PWR031" H 8750 4450 30  0001 C CNN
+F 0 "#PWR028" H 8750 4450 30  0001 C CNN
 F 1 "GND" H 8750 4380 30  0001 C CNN
 	1    8750 4450
@@
 $EndComp
 $Comp
-L +3.3V #PWR032
+L +3.3V #PWR029
 U 1 1 51728668
 P 8000 1300
-F 0 "#PWR032" H 8000 1260 30  0001 C CNN
+F 0 "#PWR029" H 8000 1260 30  0001 C CNN
 F 1 "+3.3V" H 8000 1410 30  0000 C CNN
 	1    8000 1300
@@
 $EndComp
 $Comp
-L GND #PWR033
+L GND #PWR030
 U 1 1 51728665
 P 7350 1450
-F 0 "#PWR033" H 7350 1450 30  0001 C CNN
+F 0 "#PWR030" H 7350 1450 30  0001 C CNN
 F 1 "GND" H 7350 1380 30  0001 C CNN
 	1    7350 1450
@@
 $EndComp
 $Comp
-L GND #PWR034
+L GND #PWR031
 U 1 1 51728664
 P 8650 1450
-F 0 "#PWR034" H 8650 1450 30  0001 C CNN
+F 0 "#PWR031" H 8650 1450 30  0001 C CNN
 F 1 "GND" H 8650 1380 30  0001 C CNN
 	1    8650 1450
@@
 $EndComp
 $Comp
-L +3.3V #PWR035
+L +3.3V #PWR032
 U 1 1 51728643
 P 4300 3450
-F 0 "#PWR035" H 4300 3410 30  0001 C CNN
+F 0 "#PWR032" H 4300 3410 30  0001 C CNN
 F 1 "+3.3V" H 4300 3560 30  0000 C CNN
 	1    4300 3450
@@
 $EndComp
 $Comp
-L GND #PWR036
+L GND #PWR033
 U 1 1 51728640
 P 3650 3600
-F 0 "#PWR036" H 3650 3600 30  0001 C CNN
+F 0 "#PWR033" H 3650 3600 30  0001 C CNN
 F 1 "GND" H 3650 3530 30  0001 C CNN
 	1    3650 3600
@@
 $EndComp
 $Comp
-L GND #PWR037
+L GND #PWR034
 U 1 1 5172863F
 P 4950 3600
-F 0 "#PWR037" H 4950 3600 30  0001 C CNN
+F 0 "#PWR034" H 4950 3600 30  0001 C CNN
 F 1 "GND" H 4950 3530 30  0001 C CNN
 	1    4950 3600
@@
 $EndComp
 $Comp
-L GND #PWR038
+L GND #PWR035
 U 1 1 5172861F
 P 4900 1600
-F 0 "#PWR038" H 4900 1600 30  0001 C CNN
+F 0 "#PWR035" H 4900 1600 30  0001 C CNN
 F 1 "GND" H 4900 1530 30  0001 C CNN
 	1    4900 1600
@@
 $EndComp
 $Comp
-L GND #PWR039
+L GND #PWR036
 U 1 1 5172861C
 P 3600 1600
-F 0 "#PWR039" H 3600 1600 30  0001 C CNN
+F 0 "#PWR036" H 3600 1600 30  0001 C CNN
 F 1 "GND" H 3600 1530 30  0001 C CNN
 	1    3600 1600
@@
 C_~DATAEN
 $Comp
-L +3.3V #PWR040
+L +3.3V #PWR037
 U 1 1 5158F1C7
 P 4250 1450
-F 0 "#PWR040" H 4250 1410 30  0001 C CNN
+F 0 "#PWR037" H 4250 1410 30  0001 C CNN
 F 1 "+3.3V" H 4250 1560 30  0000 C CNN
 	1    4250 1450
@@
 $EndComp
 $Comp
-L +5V #PWR041
+L +5V #PWR038
 U 1 1 5158F1A5
 P 2650 2450
-F 0 "#PWR041" H 2650 2540 20  0001 C CNN
+F 0 "#PWR038" H 2650 2540 20  0001 C CNN
 F 1 "+5V" H 2650 2540 30  0000 C CNN
 	1    2650 2450
@@
 COCO_RW
 Text HLabel 8700 4850 2    60   Output ~ 0
-ECLK
+E
 Text HLabel 10050 6350 2    60   Input ~ 0
 ~C_BUSEN
@@
 Text HLabel 4850 2000 2    60   Output ~ 0
 A0
-Text HLabel 2250 2700 2    60   Output ~ 0
+Text HLabel 2750 2700 2    60   Output ~ 0
 C_POWER
 Text Label 7400 1850 2    60   ~ 0
@@
 C_D7
 $Comp
-L GND #PWR042
+L GND #PWR039
 U 1 1 5156E804
 P 3650 2850
-F 0 "#PWR042" H 3650 2850 30  0001 C CNN
+F 0 "#PWR039" H 3650 2850 30  0001 C CNN
 F 1 "GND" H 3650 2780 30  0001 C CNN
 	1    3650 2850
@@
 $EndComp
 $Comp
-L GND #PWR043
+L GND #PWR040
 U 1 1 5156E7EC
 P 3700 4850
-F 0 "#PWR043" H 3700 4850 30  0001 C CNN
+F 0 "#PWR040" H 3700 4850 30  0001 C CNN
 F 1 "GND" H 3700 4780 30  0001 C CNN
 	1    3700 4850
@@
 C_A14
 $Comp
-L GND #PWR044
+L GND #PWR041
 U 1 1 5156E7E9
 P 7500 5700
-F 0 "#PWR044" H 7500 5700 30  0001 C CNN
+F 0 "#PWR041" H 7500 5700 30  0001 C CNN
 F 1 "GND" H 7500 5630 30  0001 C CNN
 	1    7500 5700
@@
 $EndComp
 $Comp
-L GND #PWR045
+L GND #PWR042
 U 1 1 5156E75E
 P 1950 5050
-F 0 "#PWR045" H 1950 5050 30  0001 C CNN
+F 0 "#PWR042" H 1950 5050 30  0001 C CNN
 F 1 "GND" H 1950 4980 30  0001 C CNN
 	1    1950 5050
