File: kicad/cpld.sch (KiCad schematic (older format))
At the start: 12 parts, among them P1 COCOBUS, P2 JTAG, U3 EPM3128A-TQFP144

Commit message: implement control logic for register memory
Parts:
- removed R2: 330, symbol R
- added D3: S0, symbol LED
- added D5: S1, symbol LED
- added D6: S2, symbol LED
- added JP1: CART_BOOT, symbol JUMPER
- added RP1: 150, symbol R_PACK4
Connections:
- net A_REGINT: now also U3.143 (GPIO); no longer U3.97 (GPIO)
- net C_POWER: now also RP1.5 (R4)
- net C_QCLK: now also JP1.1; no longer U3.128 (INPUT/OE2/GCLK2)
- net C_~CART: now also JP1.2; no longer U3.5 (GPIO)
- net C_~SCS: now also U3.128 (INPUT/OE2/GCLK2); no longer U3.40 (GPIO)
- net GND: now also D3.2 (K), D5.2 (K), D6.2 (K)
- net at D2.1 (A): now also RP1.4 (P4)
- net C_A15: no longer names the net of P1.39 (A15)
- net C_A15: no longer U3.44 (GPIO)
- new net: D5.1 (A), RP1.2 (P2)
- new net: D3.1 (A), RP1.1 (P1)
- new net: D6.1 (A), RP1.3 (P3)
- new net A_BUSMASTER: U3.97 (GPIO)
- new net LED0: RP1.8 (R1), U3.5 (GPIO)
- new net LED1: RP1.7 (R2), U3.44 (GPIO)
- new net LED2: RP1.6 (R3), U3.40 (GPIO)
Other:
- moved on the sheet: D2
