File: kicad/cococpld.sch (KiCad schematic (older format))
At the start: 33 parts, among them P2 JTAG, P4 TST, P5 TST, P6 TST, P7 TST, U1 LM1117-3.3, U5 EPM3032A, U6 28C256

Commit message: start of integration of common bus into CPLD
Parts:
- removed C1, C3, C4: 0.1uF, symbol C
- removed D2: A_PWR, symbol LED
- removed D3: RW, symbol LED
- removed D4: C_PWR, symbol LED
- removed D5: CTS, symbol LED
- removed D6: SCS, symbol LED
- removed D7: S0, symbol LED
- removed D8: CBUS, symbol LED
- removed JP2: SPECIAL, symbol JUMPER
- removed P2: JTAG, symbol CONN_5X2
- removed R1, R2, R3, R4, R5, R6, R7: 330, symbol R
- removed R11: 1K, symbol R
- removed R8, R9: 47K, symbol R
- removed U5: EPM3032A, symbol EPM3032A-TQFP44
- added U2: CY62256N, symbol CY62256N
Connections:
- net labels added: A_A0, A_A1, A_A10, A_A11, A_A12, A_A13, A_A14, A_A15, A_A2, A_A3, A_A4, A_A5, A_A6, A_A7, A_A8, A_A9, A_BUSREQ, A_D0, A_D1, A_D2, A_D3, A_D4, A_D5, A_D6, A_D7, A_EEN, A_REGINT, A_RW, E_~CS, M_A0, M_A1, M_A10, M_A11, M_A12, M_A13, M_A14, M_A2, M_A3, M_A4, M_A5, M_A6, M_A7, M_A8, M_A9, M_D0, M_D1, M_D2, M_D3, M_D4, M_D5, M_D6, M_D7, M_RW, M_~OE, S_~CS
- net labels removed: A0, A1, A10, A11, A12, A2, A3, A4, A5, A6, A7, A8, A9, ARD_SEL, C_POWER, C_~DATAEN, D0, D1, D2, D3, D4, D5, D6, D7, ECLK, LED_CBUS, LED_CTS, LED_RW, LED_S, LED_SCS, TCK, TDI, TDO, TMS, ~EEN, ~SCS, ~WEE
- wire segments 100 -> 4
- no-connect marks 4 -> 0
Other:
- moved on the sheet: C7, C8, C9, U1

Commit message: start of new schematic and board layout
Parts:
- removed U6: 28C256, symbol 28C256-MDS
- added C1, C10, C11, C12, C13, C3, C4, C5, C6: 0.1uF, symbol C
- added D1: S0, symbol LED
- added D2: S1, symbol LED
- added D3: S2, symbol LED
- added D4: S3, symbol LED
- added P1: COCOBUS, symbol COCOBUS
- added P2: CONN_3X2, symbol CONN_3X2
- added P3: JTAG, symbol CONN_5X2
- added RP1: 150, symbol R_PACK4
- added U3: 74LVC164245, symbol 74LVC164245
- added U4: CY62256N, symbol CY62256N
- added U5: EPM3128A-TQFP144, symbol EPM3128A-TQFP144
Connections:
- net labels added: A0, A1, A10, A11, A12, A13, A14, A2, A3, A4, A5, A6, A7, A8, A9, C_A0, C_A1, C_A10, C_A11, C_A12, C_A13, C_A14, C_A2, C_A3, C_A4, C_A5, C_A6, C_A7, C_A8, C_A9, C_D0, C_D1, C_D2, C_D3, C_D4, C_D5, C_D6, C_D7, C_ECLK, C_QCLK, C_R/~W, C_~BUSEN, C_~CART, C_~CTS, C_~HALT, C_~NMI, C_~RESET, C_~SCS, C_~SLENB, LED0, LED1, LED2, LED3, MISO, MOSI, M_~CE1, M_~CE2, M_~WE, SCLK, TCK, TDI, TDO, TMS, ~RESET
- net labels removed: A_A0, A_A1, A_A10, A_A11, A_A12, A_A13, A_A14, A_A15, A_A2, A_A3, A_A4, A_A5, A_A6, A_A7, A_A8, A_A9, A_BUSREQ, A_D0, A_D1, A_D2, A_D3, A_D4, A_D5, A_D6, A_D7, A_EEN, A_POWER, A_REGINT, A_RW, E_~CS, M_A0, M_A1, M_A10, M_A11, M_A12, M_A13, M_A14, M_A2, M_A3, M_A4, M_A5, M_A6, M_A7, M_A8, M_A9, M_RW, S_~CS
- wire segments 4 -> 80
- no-connect marks 0 -> 6
Other:
- moved on the sheet: C2, C8, C9, U1, U2

Commit message: revamped schematic
Parts:
- added C14: 0.1uF, symbol C
- added JP1: CART_BOOT, symbol JUMPER
- added U6: 50.00MHz, symbol OSC
- P2: value CONN_3X2 -> SPI; symbol CONN_3X2 -> CONN_4X2
Connections:
- net labels added: CLOCK_50, ~SS
- wire segments 80 -> 82
- no-connect marks 6 -> 7
Other:
- moved on the sheet: C2, C5, U2, U4

Commit message: updates for v1.3 board
Connections:
- net GND: no longer P2.8
- net LED0: now also RP1.1 (P1); no longer RP1.8 (R1)
- net LED1: now also RP1.2 (P2); no longer RP1.7 (R2)
- net LED2: now also RP1.3 (P3); no longer RP1.6 (R3)
- net LED3: now also RP1.4 (P4); no longer RP1.5 (R4)
- net at D1.1 (A): now also RP1.8 (R1); no longer RP1.1 (P1)
- net at D2.1 (A): now also RP1.7 (R2); no longer RP1.2 (P2)
- net at D3.1 (A): now also RP1.6 (R3); no longer RP1.3 (P3)
- net at D4.1 (A): now also RP1.5 (R4); no longer RP1.4 (P4)
- net DIRTY: now reaches U5.106 (GPIO)
- net DIRTY: now also P2.8
Changed lines of the file:
@@
-EESchema Schematic File Version 2  date 5/23/2013 7:48:54 PM
+EESchema Schematic File Version 2  date 5/25/2013 9:38:58 AM
 LIBS:power
 LIBS:device
@@
 Sheet 1 1
 Title "Color Computer Bus Interface"
-Date "23 may 2013"
+Date "25 may 2013"
 Rev "1.3"
 Comp "Bexkat Systems LLC 2013"
@@
 Comment4 ""
 $EndDescr
-NoConn ~ 4900 3500
+Wire Wire Line
+	13300 1350 13300 1400
+Wire Wire Line
+	12900 1350 13300 1350
 Wire Wire Line
 	4900 3650 4900 3750
-Connection ~ 12900 1450
-Wire Wire Line
-	12900 1500 12900 1350
 Connection ~ 4650 2450
 Wire Wire Line
@@
 Wire Wire Line
 	5950 3500 5950 3450
+Text Label 12900 1450 0    60   ~ 0
+DIRTY
+Text Label 11950 2500 0    60   ~ 0
+DIRTY
+NoConn ~ 4900 3500
 $Comp
 L +3.3V #PWR01
@@
 L GND #PWR013
 U 1 1 519E5BE3
-P 12900 1500
-F 0 "#PWR013" H 12900 1500 30  0001 C CNN
-F 1 "GND" H 12900 1430 30  0001 C CNN
-	1    12900 1500
+P 13300 1400
+F 0 "#PWR013" H 13300 1400 30  0001 C CNN
+F 1 "GND" H 13300 1330 30  0001 C CNN
+	1    13300 1400
 	1    0    0    -1
 $EndComp
@@
 F 1 "150" H 7800 7000 40  0000 C CNN
 	1    7800 7050
-	1    0    0    -1
+	-1   0    0    -1
 $EndComp
 Text Label 4850 6850 0    60   ~ 0

Commit message: minor edits
Parts:
- removed C1, C3, C4, C6: 0.1uF, symbol C
- removed U3: 74LVC164245, symbol 74LVC164245
Connections:
- net C_~BUSEN: no longer names the net of U5.74 (GPIO)
Changed lines of the file:
@@
-EESchema Schematic File Version 2  date 5/25/2013 9:38:58 AM
+EESchema Schematic File Version 2  date 5/26/2013 11:02:39 AM
 LIBS:power
 LIBS:device
@@
 Sheet 1 1
 Title "Color Computer Bus Interface"
-Date "25 may 2013"
+Date "26 may 2013"
 Rev "1.3"
 Comp "Bexkat Systems LLC 2013"
@@
 Comment4 ""
 $EndDescr
+Text Label 4150 2150 0    60   ~ 0
+C_A14
+Text Label 4150 2050 0    60   ~ 0
+C_A13
+Text Label 4150 1950 0    60   ~ 0
+C_A12
+Text Label 4150 1850 0    60   ~ 0
+C_A11
+Text Label 4150 1750 0    60   ~ 0
+C_A10
+Text Label 4150 1650 0    60   ~ 0
+C_A9
+Text Label 4150 1550 0    60   ~ 0
+C_A8
+Text Label 4150 1450 0    60   ~ 0
+C_A7
+Text Label 4150 1350 0    60   ~ 0
+C_A6
+Text Label 4150 1250 0    60   ~ 0
+C_A5
+Text Label 4150 1150 0    60   ~ 0
+C_A4
+Text Label 4150 1050 0    60   ~ 0
+C_A3
+Text Label 4150 950  0    60   ~ 0
+C_A2
+Text Label 4150 850  0    60   ~ 0
+C_A1
+Text Label 4150 750  0    60   ~ 0
+C_A0
 Wire Wire Line
 	13300 1350 13300 1400
@@
 Wire Wire Line
 	4900 3650 4900 3750
-Connection ~ 4650 2450
-Wire Wire Line
-	4650 2350 4650 2550
-Wire Wire Line
-	2400 2550 2400 2450
-Connection ~ 2950 1100
-Connection ~ 3050 1100
-Wire Wire Line
-	3100 1100 2900 1100
-Wire Wire Line
-	3050 1100 3050 1300
-Wire Wire Line
-	2500 1150 2500 1100
 Wire Wire Line
 	7250 6650 7350 6650
@@
 	2050 7750 2050 7550
 Connection ~ 2050 7650
-Wire Wire Line
-	3500 1100 3500 1150
-Wire Wire Line
-	2950 1100 2950 1300
-Wire Wire Line
-	3000 1000 3000 1100
-Connection ~ 3000 1100
-Connection ~ 5250 1100
-Wire Wire Line
-	5250 1000 5250 1100
-Wire Wire Line
-	5200 1100 5200 1300
-Wire Wire Line
-	5750 1100 5750 1150
-Wire Wire Line
-	4750 1150 4750 1100
-Wire Wire Line
-	5300 1100 5300 1300
-Wire Wire Line
-	5350 1100 5150 1100
-Connection ~ 5300 1100
-Connection ~ 5200 1100
 Wire Wire Line
 	5950 3500 5950 3450
@@
 Text Label 1950 6500 0    60   ~ 0
 C_~CART
-Text Label 11950 5200 0    60   ~ 0
-C_~BUSEN
 Text Label 3650 4400 0    60   ~ 0
 M_~CE2
@@
 Text Label 1200 3300 0    60   ~ 0
 C_A0
-Text Label 4650 2250 2    60   ~ 0
-C_A14
-Text Label 4650 2150 2    60   ~ 0
-C_A13
-Text Label 4650 2050 2    60   ~ 0
-C_A12
-Text Label 4650 1950 2    60   ~ 0
-C_A11
-Text Label 4650 1850 2    60   ~ 0
-C_A10
-Text Label 4650 1750 2    60   ~ 0
-C_A9
-Text Label 4650 1650 2    60   ~ 0
-C_A8
-Text Label 2400 2350 2    60   ~ 0
-C_A7
-Text Label 2400 2250 2    60   ~ 0
-C_A6
-Text Label 2400 2150 2    60   ~ 0
-C_A5
-Text Label 2400 2050 2    60   ~ 0
-C_A4
-Text Label 2400 1950 2    60   ~ 0
-C_A3
-Text Label 2400 1850 2    60   ~ 0
-C_A2
-Text Label 2400 1750 2    60   ~ 0
-C_A1
-Text Label 2400 1650 2    60   ~ 0
-C_A0
-Text Label 5850 2250 0    60   ~ 0
-A14
-Text Label 5850 2150 0    60   ~ 0
-A13
-Text Label 5850 2050 0    60   ~ 0
-A12
-Text Label 5850 1950 0    60   ~ 0
-A11
-Text Label 5850 1850 0    60   ~ 0
-A10
-Text Label 5850 1750 0    60   ~ 0
-A9
-Text Label 5850 1650 0    60   ~ 0
-A8
-Text Label 3600 2350 0    60   ~ 0
-A7
-Text Label 3600 2250 0    60   ~ 0
-A6
-Text Label 3600 2150 0    60   ~ 0
-A5
-Text Label 3600 2050 0    60   ~ 0
-A4
-Text Label 3600 1950 0    60   ~ 0
-A3
-Text Label 3600 1850 0    60   ~ 0
-A2
-Text Label 3600 1750 0    60   ~ 0
-A1
-Text Label 3600 1650 0    60   ~ 0
-A0
-Text Label 5850 2450 0    60   ~ 0
-C_~BUSEN
-Text Label 3600 2450 0    60   ~ 0
-C_~BUSEN
-$Comp
-L GND #PWR05
-U 1 1 519E5CD9
-P 2400 2550
-F 0 "#PWR05" H 2400 2550 30  0001 C CNN
-F 1 "GND" H 2400 2480 30  0001 C CNN
-	1    2400 2550
-	1    0    0    -1
-$EndComp
-$Comp
-L GND #PWR06
-U 1 1 519E5CD6
-P 4650 2550
-F 0 "#PWR06" H 4650 2550 30  0001 C CNN
-F 1 "GND" H 4650 2480 30  0001 C CNN
-	1    4650 2550
-	1    0    0    -1
-$EndComp
-$Comp
-L 74LVC164245 U3
-U 2 1 519E5CBA
-P 5250 2000
-F 0 "U3" H 5500 2550 60  0000 C CNN
-F 1 "74LVC164245" H 5250 1400 60  0000 C CNN
-	2    5250 2000
-	1    0    0    -1
-$EndComp
-$Comp
-L C C6
-U 1 1 519E5CB9
-P 5550 1100
-F 0 "C6" H 5600 1200 50  0000 L CNN
-F 1 "0.1uF" H 5600 1000 50  0000 L CNN
-	1    5550 1100
-	0    -1   -1   0
-$EndComp
-$Comp
-L C C4
-U 1 1 519E5CB8
-P 4950 1100
-F 0 "C4" H 5000 1200 50  0000 L CNN
-F 1 "0.1uF" H 5000 1000 50  0000 L CNN
-	1    4950 1100
-	0    -1   -1   0
-$EndComp
-$Comp
-L GND #PWR07
-U 1 1 519E5CB7
-P 5750 1150
-F 0 "#PWR07" H 5750 1150 30  0001 C CNN
-F 1 "GND" H 5750 1080 30  0001 C CNN
-	1    5750 1150
-	-1   0    0    -1
-$EndComp
-$Comp
-L GND #PWR08
-U 1 1 519E5CB6
-P 4750 1150
-F 0 "#PWR08" H 4750 1150 30  0001 C CNN
-F 1 "GND" H 4750 1080 30  0001 C CNN
-	1    4750 1150
-	-1   0    0    -1
-$EndComp
-$Comp
-L +3.3V #PWR09
-U 1 1 519E5CB5
-P 5250 1000
-F 0 "#PWR09" H 5250 960 30  0001 C CNN
-F 1 "+3.3V" H 5250 1110 30  0000 C CNN
-	1    5250 1000
-	-1   0    0    -1
-$EndComp
-$Comp
-L +3.3V #PWR010
-U 1 1 519E5C9B
-P 3000 1000
-F 0 "#PWR010" H 3000 960 30  0001 C CNN
-F 1 "+3.3V" H 3000 1110 30  0000 C CNN
-	1    3000 1000
-	-1   0    0    -1
-$EndComp
-$Comp
-L GND #PWR011
-U 1 1 519E5C84
-P 2500 1150
-F 0 "#PWR011" H 2500 1150 30  0001 C CNN
-F 1 "GND" H 2500 1080 30  0001 C CNN
-	1    2500 1150
-	-1   0    0    -1
-$EndComp
-$Comp
-L GND #PWR012
-U 1 1 519E5C7D
-P 3500 1150
-F 0 "#PWR012" H 3500 1150 30  0001 C CNN
-F 1 "GND" H 3500 1080 30  0001 C CNN
-	1    3500 1150
-	-1   0    0    -1
-$EndComp
-$Comp
-L C C1
-U 1 1 519E5C6F
-P 2700 1100
-F 0 "C1" H 2750 1200 50  0000 L CNN
-F 1 "0.1uF" H 2750 1000 50  0000 L CNN
-	1    2700 1100
-	0    -1   -1   0
-$EndComp
-$Comp
-L C C3
-U 1 1 519E5C67
-P 3300 1100
-F 0 "C3" H 3350 1200 50  0000 L CNN
-F 1 "0.1uF" H 3350 1000 50  0000 L CNN
-	1    3300 1100
-	0    -1   -1   0
-$EndComp
-$Comp
-L 74LVC164245 U3
-U 1 1 519E5C5A
-P 3000 2000
-F 0 "U3" H 3250 2550 60  0000 C CNN
-F 1 "74LVC164245" H 3000 1400 60  0000 C CNN
-	1    3000 2000
-	1    0    0    -1
-$EndComp
 Text Label 11200 1700 1    60   ~ 0
 MOSI

Commit message: start to change memory and bus config
Parts:
- removed C5: 0.1uF, symbol C
- removed U2, U4: CY62256N, symbol CY62256N
- added U?: R1LP0108ESF-5SI, symbol R1LP0108ESF-5SI
Connections:
- net +3.3V: now also C2.1, U?.6 (CS2), U?.8 (Vcc)
- net +5V: no longer C2.1
- net A0: now also U?.20 (A0)
- net A1: now also U?.19 (A1)
- net A10: now also U?.31 (A10)
- net A11: now also U?.1 (A11)
- net A12: now also U?.12 (A12)
- net A13: now also U?.4 (A13)
- net A14: now also U?.11 (A14)
- net A2: now also U?.18 (A2)
- net A3: now also U?.17 (A3)
- net A4: now also U?.16 (A4)
- net A5: now also U?.15 (A5)
- net A6: now also U?.14 (A6)
- net A7: now also U?.13 (A7)
- net A8: now also U?.3 (A8)
- net A9: now also U?.2 (A9)
- net GND: now also U?.24 (GND)
- net M_D0: now also U?.21 (D0)
- net M_D1: now also U?.22 (D1)
- net M_D2: now also U?.23 (D2)
- net M_D3: now also U?.25 (D3)
- net M_D4: now also U?.26 (D4)
- net M_D5: now also U?.27 (D5)
- net M_D6: now also U?.28 (D6)
- net M_D7: now also U?.29 (D7)
- net M_~OE: now also U?.32 (~OE)
- net M_~WE: now also U?.5 (~WE)
- net A15: now reaches U5.44 (GPIO)
- net A15: now also U?.7 (A15)
- net M_~CE1 renamed M_~CE
- net M_~CE: now also U?.30 (~CS1)
- net M_~CE2: no longer names the net of U5.63 (GPIO)
- new net A16: U?.10 (A16)

Commit message: v1.4 HW design
Parts:
- removed C12, C13: 0.1uF, symbol C
- removed U1: LM1117-3.3, symbol LM1117-3.3
- added D5: DIODE, symbol DIODE
- added U1: TLV1117-33, symbol TLV1117-33
- C9: value 10uF -> 100uF
- U5: value EPM3128A-TQFP144 -> EPM3256A-TQFP144
- gave numbers to parts that had none: 1
Connections:
- net A16 is gone; now on net +3.3V: U2.10 (A16)
- net C_A0 is gone; now on net A0: P1.19 (A0)
- net C_A1 is gone; now on net A1: P1.20 (A1)
- net C_A10 is gone; now on net A10: P1.29 (A10)
- net C_A11 is gone; now on net A11: P1.30 (A11)
- net C_A12 is gone; now on net A12: P1.31 (A12)
- net C_A13 is gone; now on net A13: P1.37 (A13)
- net C_A14 is gone; now on net A14: P1.38 (A14)
- net C_A2 is gone; now on net A2: P1.21 (A2)
- net C_A3 is gone; now on net A3: P1.22 (A3)
- net C_A4 is gone; now on net A4: P1.23 (A4)
- net C_A5 is gone; now on net A5: P1.24 (A5)
- net C_A6 is gone; now on net A6: P1.25 (A6)
- net C_A7 is gone; now on net A7: P1.26 (A7)
- net C_A8 is gone; now on net A8: P1.27 (A8)
- net C_A9 is gone; now on net A9: P1.28 (A9)
- net +3.3V: now also D5.1 (A), U1.2 (VO)
- net +5V: now also D5.2 (K), U1.3 (VI)
- net GND: now also U1.1 (GND)
Other:
- moved on the sheet: C2, C8, C9, JP1, U2
