File: kicad/Coco.sch (KiCad schematic (older format))
At the start: 11 parts

Commit message: hardware prototype for v2.0 board
Parts:
- removed P?: JTAG, symbol CONN_5X2
- added D1: S0, symbol LED
- added D2: S1, symbol LED
- added D3: S2, symbol LED
- added D4: S3, symbol LED
- added R2: 47k, ~, symbol R
- added RP1: 150, symbol R_PACK4
- added SW1: CART_BOOT, ~, symbol SWITCH_INV
- gave numbers to parts that had none: 10
Connections:
- net ~SS is gone; now on net M_D6: U2.38 (GPIO)
- net A_A0: now also U2.98 (GPIO)
- net A_A1: now also U2.16 (GPIO)
- net A_A10: now also U2.131 (GPIO)
- net A_A11: now also U2.15 (GPIO)
- net A_A12: now also U2.132 (GPIO)
- net A_A13: now also U2.62 (GPIO)
- net A_A14: now also U2.79 (GPIO)
- net A_A15: now also U2.103 (GPIO)
- net A_A2: now also U2.10 (GPIO)
- net A_A3: now also U2.92 (GPIO)
- net A_A4: now also U2.109 (GPIO)
- net A_A5: now also U2.69 (GPIO)
- net A_A6: now also U2.54 (GPIO)
- net A_A7: now also U2.81 (GPIO)
- net A_A8: now also U2.140 (GPIO)
- net A_A9: now also U2.66 (GPIO)
- net A_D0: now also U2.113 (GPIO)
- net A_D1: now also U2.116 (GPIO)
- net A_D2: now also U2.117 (GPIO)
- net A_D3: now also U2.118 (GPIO)
- net A_D4: now also U2.119 (GPIO)
- net A_D5: now also U2.120 (GPIO)
- net A_D6: now also U2.121 (GPIO)
- net A_D7: now also U2.122 (GPIO)
- net A_R/~W: now also U2.63 (GPIO)
- net A_~SELECT: now also U2.83 (GPIO)
- net C_A0: now also U2.23 (GPIO); no longer U2.65 (GPIO)
- net C_A1: now also U2.139 (GPIO); no longer U2.81 (GPIO)
- net C_A10: now also U2.12 (GPIO); no longer U2.72 (GPIO)
- net C_A11: now also U2.47 (GPIO); no longer U2.132 (GPIO)
- net C_A12: now also U2.110 (GPIO); no longer U2.84 (GPIO)
- net C_A13: now also U2.78 (GPIO); no longer U2.11 (GPIO)
- net C_A14: now also U2.102 (GPIO); no longer U2.37 (GPIO)
- net C_A3: now also U2.53 (GPIO); no longer U2.40 (GPIO)
- net C_A4: now also U2.65 (GPIO); no longer U2.45 (GPIO)
- net C_A5: now also U2.91 (GPIO); no longer U2.113 (GPIO)
- net C_A6: now also U2.133 (GPIO); no longer U2.112 (GPIO)
- net C_A7: now also U2.5 (GPIO); no longer U2.131 (GPIO)
- net C_A8: now also U2.71 (GPIO); no longer U2.29 (GPIO)
- net C_A9: now also U2.111 (GPIO); no longer U2.91 (GPIO)
- net C_D0: now also U2.28 (GPIO); no longer U2.22 (GPIO)
- net C_D1: now also U2.29 (GPIO); no longer U2.23 (GPIO)
- net C_D2: now also U2.30 (GPIO); no longer U2.21 (GPIO)
- net C_D3: now also U2.31 (GPIO); no longer U2.122 (GPIO)
- net C_D4: now also U2.32 (GPIO); no longer U2.121 (GPIO)
- net C_D5: now also U2.34 (GPIO); no longer U2.117 (GPIO)
- net C_D6: now also U2.35 (GPIO); no longer U2.31 (GPIO)
- net C_ECLK: now also U2.86 (GPIO); no longer U2.12 (GPIO)
- net C_POWER: now also U2.9 (GPIO), R2.1; no longer U2.2 (GPIO)
- net C_QCLK: now also SW1.2; no longer U2.5 (GPIO)
- net C_R/~W: now also U2.48 (GPIO); no longer U2.79 (GPIO)
- net C_~CART: now also SW1.1; no longer U2.8 (GPIO)
- net C_~CTS: now also U2.11 (GPIO); no longer U2.103 (GPIO)
- net C_~HALT: now also U2.100 (GPIO); no longer U2.136 (GPIO)
- net C_~NMI: now also U2.90 (GPIO); no longer U2.7 (GPIO)
- net C_~RESET: no longer U2.127 (INPUT/GCLRn)
- net C_~SCS: now also U2.106 (GPIO); no longer U2.75 (GPIO)
- net C_~SLENB: now also U2.1 (GPIO); no longer U2.19 (GPIO)
- net GND: now also D1.2 (K), D2.2 (K), D3.2 (K), D4.2 (K), R2.2
- net LED0: now also U2.99 (GPIO), RP1.1 (P1); no longer U2.54 (GPIO)
- net LED1: now also U2.138 (GPIO), RP1.2 (P2); no longer U2.139 (GPIO)
- net LED2: now also U2.136 (GPIO), RP1.3 (P3); no longer U2.140 (GPIO)
- net LED3: now also U2.143 (GPIO), RP1.4 (P4); no longer U2.141 (GPIO)
- net M_A0: now also U2.74 (GPIO); no longer U2.53 (GPIO)
- net M_A1: now also U2.68 (GPIO); no longer U2.49 (GPIO)
- net M_A10: now also U2.75 (GPIO); no longer U2.16 (GPIO)
- net M_A11: now also U2.60 (GPIO); no longer U2.18 (GPIO)
- net M_A12: now also U2.56 (GPIO); no longer U2.138 (GPIO)
- net M_A13: now also U2.55 (GPIO); no longer U2.137 (GPIO)
- net M_A14: now also U2.18 (GPIO); no longer U2.34 (GPIO)
- net M_A15: now also U2.19 (GPIO); no longer U2.35 (GPIO)
- net M_A2: now also U2.22 (GPIO); no longer U2.99 (GPIO)
- net M_A3: now also U2.25 (GPIO); no longer U2.56 (GPIO)
- net M_A4: now also U2.27 (GPIO); no longer U2.63 (GPIO)
- net M_A5: now also U2.21 (GPIO); no longer U2.88 (GPIO)
- net M_A6: now also U2.88 (GPIO); no longer U2.87 (GPIO)
- net M_A7: now also U2.87 (GPIO); no longer U2.62 (GPIO)
- net M_A8: now also U2.84 (GPIO); no longer U2.134 (GPIO)
- net M_A9: now also U2.82 (GPIO); no longer U2.28 (GPIO)
- net M_D0: now also U2.44 (GPIO); no longer U2.46 (GPIO)
- net M_D1: now also U2.43 (GPIO); no longer U2.25 (GPIO)
- net M_D2: now also U2.42 (GPIO); no longer U2.27 (GPIO)
- net M_D3: now also U2.41 (GPIO); no longer U2.120 (GPIO)
- net M_D4: now also U2.40 (GPIO); no longer U2.118 (GPIO)
- net M_D5: now also U2.39 (GPIO); no longer U2.116 (GPIO)
- net M_D6: no longer U2.92 (GPIO)
- net M_D7: now also U2.37 (GPIO); no longer U2.96 (GPIO)
- net M_~CE: now also U2.142 (GPIO); no longer U2.100 (GPIO)
- net M_~OE: now also U2.2 (GPIO); no longer U2.48 (GPIO)
- net M_~WE: now also U2.112 (GPIO); no longer U2.32 (GPIO)
- net SCLK_33: now reaches U2.101 (GPIO)
- net MOSI: now reaches U2.107 (GPIO)
- net MOSI_33: now reaches U2.61 (GPIO)
- net SD_SS: now reaches U2.67 (GPIO)
- new net: D4.1 (A), RP1.5 (R4)
- new net: D2.1 (A), RP1.7 (R2)
- new net: D1.1 (A), RP1.8 (R1)
- new net: D3.1 (A), RP1.6 (R3)
- new net A_FCFG_I: U2.134 (GPIO)
- new net A_FCMD_I: U2.137 (GPIO)
- new net SCLK: U2.72 (GPIO)
- new net SD_SS_33: U2.49 (GPIO)
- new net ~RESET: U2.127 (INPUT/GCLRn)
- no-connect marks 6 -> 3

Commit message: possible v2.1 design changes
Connections:
- net GND: now also U5.30 (~CS1)
- net M_~CE: no longer names the net of U2.142 (GPIO)
- net M_~CE: no longer U5.30 (~CS1)
Changed lines of the file:
@@
 Sheet 2 3
 Title "Color Computer FDC Ethernet Controller"
-Date "25 aug 2013"
+Date "10 sep 2013"
 Rev "2.1"
 Comp "Bexkat Systems LLC 2013"
@@
 Text Label 3850 1500 1    60   ~ 0
 LED3
-Text Label 3950 1500 1    60   ~ 0
-M_~CE
 Text Label 6950 1500 1    60   ~ 0
 M_~WE
@@
 	-1   0    0    -1
 $EndComp
-Text Label 12000 1600 0    60   ~ 0
-M_~CE
 $Comp
 L R1LP0108ESF-5SI U5
@@
 Text HLabel 5450 1500 1    60   Input ~ 0
 ~RESET
+$Comp
+L GND #PWR?
+U 1 1 522E6ECC
+P 12400 1700
+F 0 "#PWR?" H 12400 1700 30  0001 C CNN
+F 1 "GND" H 12400 1630 30  0001 C CNN
+F 2 "" H 12400 1700 60  0001 C CNN
+F 3 "" H 12400 1700 60  0001 C CNN
+	1    12400 1700
+	1    0    0    -1
+$EndComp
+Wire Wire Line
+	12000 1600 12400 1600
+Wire Wire Line
+	12400 1600 12400 1700
 $EndSCHEMATC
